File: preamp.kicad_sch (KiCad schematic)
At the start: 12 parts, among them U2 OPA357AIDBVR, U7 LM4040AIM3-3.0+T

Commit message: Updated BOM, schematic , foortprints, symbols
Parts:
- R2, R4: footprint ERJ3EKF2103V:RES_ERJ3EKF2103V -> ERJ3EKF1001V:RES_ERJ3EKF1001V
- R5: footprint ERJ3EKF2103V:RES_ERJ3EKF2103V -> ERJ3EKF1000V:RES_ERJ3EKF1000V
- R6: footprint ERJ3EKF2103V:RES_ERJ3EKF2103V -> ERJ3EKF2101V:RES_ERJ3EKF2101V
Changed lines of the file:
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@@
 		(title "Amplifier")
 		(date "2025-03-23")
-		(rev "0.1.1")
+		(rev "0.1.2")
 		(company "Vadym Vikulin")
 	)
@@
 			)
 		)
-		(property "Footprint" "ERJ3EKF2103V:RES_ERJ3EKF2103V"
+		(property "Footprint" "ERJ3EKF1001V:RES_ERJ3EKF1001V"
 			(at 80.01 85.598 90)
 			(effects
@@
 			)
 		)
-		(property "Footprint" "ERJ3EKF2103V:RES_ERJ3EKF2103V"
+		(property "Footprint" "ERJ3EKF2101V:RES_ERJ3EKF2101V"
 			(at 119.38 70.358 90)
 			(effects
@@
 			)
 		)
-		(property "Footprint" "ERJ3EKF2103V:RES_ERJ3EKF2103V"
+		(property "Footprint" "ERJ3EKF1000V:RES_ERJ3EKF1000V"
 			(at 80.01 95.758 90)
 			(effects
@@
 			)
 		)
-		(property "Footprint" "ERJ3EKF2103V:RES_ERJ3EKF2103V"
+		(property "Footprint" "ERJ3EKF1001V:RES_ERJ3EKF1001V"
 			(at 74.168 100.33 90)
 			(effects

Commit message: Removed VR2 resistor and adjusted R6 to prevent self-oscillation of the amplifier
Parts:
- removed VR2: 5k, 3296W-1-502LF:TRIM_3296W-1-502LF, symbol 3296W-1-502LF-1:3296W-1-502LF_1
- R6: value 2.1k -> 1k; footprint ERJ3EKF2101V:RES_ERJ3EKF2101V -> ERJ3EKF1001V:RES_ERJ3EKF1001V
Other:
- moved on the sheet: R6

Commit message: Updated BOM format accordingly to PCBWay format
Parts:
- C4: MP (none) -> CL10A226MP8NUNE; Package (none) -> 0603 Samsung
- D1: MP (none) -> 933976380215; Package (none) -> SOT-23
- R1, R3: MP (none) -> ERJ3EKF2103V; Package (none) -> 0603
- R2, R4, R6: MP (none) -> ERJ3EKF1001V; Package (none) -> 0603
- R5: MP (none) -> ERJ3EKF1000V; Package (none) -> 0603
Changed lines of the file:
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@@
+			)
+		)
+		(property "MP" "ERJ3EKF1001V"
+			(at 80.01 83.82 0)
+			(effects
+				(font
+					(size 1.27 1.27)
+				)
+				(hide yes)
+			)
+		)
+		(property "Package" "0603"
+			(at 80.01 83.82 0)
+			(effects
+				(font
+					(size 1.27 1.27)
+				)
+				(hide yes)
 			)
 		)
@@
 			)
 		)
+		(property "MP" "ERJ3EKF1001V"
+			(at 110.49 68.58 0)
+			(effects
+				(font
+					(size 1.27 1.27)
+				)
+				(hide yes)
+			)
+		)
+		(property "Package" "0603"
+			(at 110.49 68.58 0)
+			(effects
+				(font
+					(size 1.27 1.27)
+				)
+				(hide yes)
+			)
+		)
 		(pin "2"
 		)
@@
 		)
 		(property "Description" "Resistor"
+			(at 68.58 72.39 0)
+			(effects
+				(font
+					(size 1.27 1.27)
+				)
+				(hide yes)
+			)
+		)
+		(property "MP" "ERJ3EKF2103V"
+			(at 68.58 72.39 0)
+			(effects
+				(font
+					(size 1.27 1.27)
+				)
+				(hide yes)
+			)
+		)
+		(property "Package" "0603"
 			(at 68.58 72.39 0)
 			(effects
@@
 			)
 		)
+		(property "MP" "CL10A226MP8NUNE"
+			(at 104.14 109.22 0)
+			(effects
+				(font
+					(size 1.27 1.27)
+				)
+				(hide yes)
+			)
+		)
+		(property "Package" "0603 Samsung"
+			(at 104.14 109.22 0)
+			(effects
+				(font
+					(size 1.27 1.27)
+				)
+				(hide yes)
+			)
+		)
 		(pin "2"
 		)
@@
 			)
 		)
+		(property "Package" "SOT-23"
+			(at 87.63 102.87 0)
+			(effects
+				(font
+					(size 1.27 1.27)
+				)
+				(hide yes)
+			)
+		)
+		(property "MP" "933976380215"
+			(at 87.63 102.87 0)
+			(effects
+				(font
+					(size 1.27 1.27)
+				)
+				(hide yes)
+			)
+		)
 		(pin "1"
 		)
@@
 			)
 		)
+		(property "MP" "ERJ3EKF1000V"
+			(at 80.01 93.98 0)
+			(effects
+				(font
+					(size 1.27 1.27)
+				)
+				(hide yes)
+			)
+		)
+		(property "Package" "0603"
+			(at 80.01 93.98 0)
+			(effects
+				(font
+					(size 1.27 1.27)
+				)
+				(hide yes)
+			)
+		)
 		(pin "2"
 		)
@@
 		)
 		(property "Description" "Resistor"
+			(at 76.2 72.39 0)
+			(effects
+				(font
+					(size 1.27 1.27)
+				)
+				(hide yes)
+			)
+		)
+		(property "MP" "ERJ3EKF2103V"
+			(at 76.2 72.39 0)
+			(effects
+				(font
+					(size 1.27 1.27)
+				)
+				(hide yes)
+			)
+		)
+		(property "Package" "0603"
 			(at 76.2 72.39 0)
 			(effects
@@
 			(at 72.39 100.33 0)
 			(effects
+				(font
+					(size 1.27 1.27)
+				)
+				(hide yes)
+			)
+		)
+		(property "MP" "ERJ3EKF1001V"
+			(at 72.39 100.33 0)
+			(effects
+				(font
+					(size 1.27 1.27)
+				)
+				(hide yes)
+			)
+		)
+		(property "Package" "0603"
+			(at 72.39 100.33 0)
+			(effects
