File: sipm_board.kicad_sch (KiCad schematic)
At the start: 15 parts, among them Q2 MMBT5088LT1G, Q3 MMBT5088LT1G, U10 MICROFC-60035-SMT-TR1, U9 TPS7B6950DBVR

Commit message: 3d models update
Parts:
- renumbered TH2 to TH1
Changed lines of the file:
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@@
 	(title_block
 		(title "SiPM Board")
-		(date "2025-09-06")
-		(rev "0.2.1")
+		(date "2025-09-07")
+		(rev "0.2.3")
 		(company "Vadym Vikulin")
 		(comment 7 "Temperature Correction (~21 mV/K)")
@@
 		(on_board yes)
 		(dnp no)
-		(property "Reference" "TH2"
+		(property "Reference" "TH1"
 			(at 127.254 76.962 0)
 			(effects
@@
 		(pin "2"
 		)
+		(instances
+			(project "gamma-spectrometer"
+				(path "/1fc9c372-472b-46ca-8d3b-f4aefe31a8be/1929b78d-718a-49ce-a44a-01f5c50b8f35"
+					(reference "TH1")
+					(unit 1)
+				)
+			)
+		)
 	)
 	(symbol
@@
 		(pin "5"
 		)
+		(instances
+			(project "gamma-spectrometer"
+				(path "/1fc9c372-472b-46ca-8d3b-f4aefe31a8be/1929b78d-718a-49ce-a44a-01f5c50b8f35"
+					(reference "U10")
+					(unit 1)
+				)
+			)
+		)
 	)
 	(symbol
@@
 		(pin "5"
 		)
+		(instances
+			(project "gamma-spectrometer"
+				(path "/1fc9c372-472b-46ca-8d3b-f4aefe31a8be/1929b78d-718a-49ce-a44a-01f5c50b8f35"
+					(reference "U9")
+					(unit 1)
+				)
+			)
+		)
 	)
