File: amplifier.kicad_sch (KiCad schematic)
At the start: 15 parts, among them T1 T1-1T-KK81, U5 LM4040AIM3, U8 OPA357AIDBVR

Commit message: Title fix
Other:
- title: SiPM Board -> Amplifier
Changed lines of the file:
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@@
 	(paper "A4")
 	(title_block
-		(title "SiPM Board")
+		(title "Amplifier")
 		(date "2025-09-06")
-		(rev "0.2.1")
+		(rev "0.2.2")
 		(company "Vadym Vikulin")
 		(comment 7 "Temperature Correction (~21 mV/K)")
