File: modules/OGK-Motherboard/amplifier.kicad_sch (KiCad schematic)
At the start: 15 parts, among them T1 T1-1T-KK81, U5 LM4040AIM3, U8 OPA357AIDBVR

Commit message: Modular motherboard
Parts:
- renumbered C33 to C20, C20 to C21, C21 to C22, R2 to R1, R22 to R11, R23 to R12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
